File: breakout proto.sch (EAGLE design)
At the start: 50 parts, among them SW1 SPST_TACT-KMR2, U1 MCU-ATSAMD51J, Y1 32.768

Commit message: Add files via upload
Parts:
- removed _: USB-C-CON-MIDBRD-SHORT-1-2295018-2EXTEN, 0TG-Lib v01.3:USB-C-CON-MIDBRD-SHORT-1-2295018-2EXTEN
- added U$17: USB-C-PCB-USB-2.0-TYPE-CDS_3, 0TG-Lib v01.3:USB-C-PCB-USB-2.0-TYPE-CDS_3
Connections:
- net D+: now also U$17.D-; no longer _.A_D+, _.B_D+
- net D-: now also U$17.D+; no longer _.A_D-, _.B_D-
- net GND: now also U$17.GND; no longer _.A_GND1, _.A_GND2, _.B_GND1, _.B_GND2, _.SHIELD
- net VBUS_RAW: now also U$17.VBUS; no longer _.A_VBUS1, _.A_VBUS2, _.B_VBUS1, _.B_VBUS2
Other:
- moved on the sheet: F1
